File: Left/left.kicad_sch (KiCad schematic)
At the start: 215 parts, among them J1 USB_EXT, J2 USB_Conn_1, J3 USB_Link, J4 Conn_01x06, J5 JTAG_TC2030, J6 USB_Conn_2, Q1 MUN5311DW1T1G, Q2 AO3401A, Q3 MUN5311DW1T1G, SW1 Reset, T1 TP, T10 TP, T11 TP, T12 TP, T13 TP, T14 TP, T15 TP, T16 TP, T17 TP, T18 TP, T19 TP, T2 TP, T20 TP, T21 TP, T22 TP, T23 TP, T24 3V3, T25 5V, T26 GND, T27 GND, T3 TP, T4 TP, T5 TP, T6 TP, T7 TP, T8 TP, T9 TP, U1 TS3A27518ERTW, U2 SRV05-4, U3 STM32F411CEU6, U4 MB85RS64PNF-G-JNERE1, U5 AAP2967-33VIR1, U6 LMV321, U7 W25Q128JVSIQ, U8 SN74LV1T34DCKR, Y1 SMD-CRYSTAL-8MHZ-20PF-10PPM_2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

Commit message: Before rotating switches and LEDs...
Connections:
- net FLASH_CS: now also U3.31 (PA10); no longer U3.11 (PA1)
- net RGB_DATA: now also U3.11 (PA1); no longer U3.31 (PA10)
Other:
- moved on the sheet: R5
Changed lines of the file:
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@@
   (junction (at 62.23 181.61) (diameter 0) (color 0 0 0 0)
   )
+  (junction (at 101.6 105.41) (diameter 0) (color 0 0 0 0)
+  )
   (junction (at 541.02 96.52) (diameter 0) (color 0 0 0 0)
   )
@@
   (junction (at 198.12 90.17) (diameter 0) (color 0 0 0 0)
   )
-  (junction (at 101.6 128.27) (diameter 0) (color 0 0 0 0)
-  )
   (junction (at 180.34 165.1) (diameter 0) (color 0 0 0 0)
   )
@@
     (stroke (width 0) (type default) (color 0 0 0 0))
   )
-  (wire (pts (xy 82.55 128.27) (xy 101.6 128.27))
-    (stroke (width 0) (type default) (color 0 0 0 0))
-  )
   (wire (pts (xy 66.04 354.33) (xy 66.04 351.79))
     (stroke (width 0) (type default) (color 0 0 0 0))
@@
     (stroke (width 0) (type default) (color 0 0 0 0))
   )
+  (wire (pts (xy 82.55 128.27) (xy 93.98 128.27))
+    (stroke (width 0) (type default) (color 0 0 0 0))
+  )
   (wire (pts (xy 138.43 102.87) (xy 157.48 102.87))
     (stroke (width 0) (type default) (color 0 0 0 0))
@@
     (stroke (width 0) (type default) (color 0 0 0 0))
   )
-  (wire (pts (xy 82.55 105.41) (xy 93.98 105.41))
-    (stroke (width 0) (type default) (color 0 0 0 0))
-  )
   (wire (pts (xy 411.48 295.91) (xy 398.78 295.91))
     (stroke (width 0) (type default) (color 0 0 0 0))
@@
     (stroke (width 0) (type default) (color 0 0 0 0))
   )
+  (wire (pts (xy 82.55 105.41) (xy 101.6 105.41))
+    (stroke (width 0) (type default) (color 0 0 0 0))
+  )
   (polyline (pts (xy 200.66 270.51) (xy 15.24 270.51))
     (stroke (width 0) (type default) (color 0 0 0 0))
@@
     (stroke (width 0) (type default) (color 0 0 0 0))
   )
-  (wire (pts (xy 101.6 128.27) (xy 114.3 128.27))
+  (wire (pts (xy 101.6 105.41) (xy 114.3 105.41))
     (stroke (width 0) (type default) (color 0 0 0 0))
   )
@@
   )
   (text "Pullup hack to be able to use\n3.3V logic for 5V input of RGB LED"
-    (at 95.25 133.35 0)
+    (at 95.25 110.49 0)
     (effects (font (size 1.27 1.27)) (justify left bottom))
   )
@@
     (effects (font (size 1.27 1.27)) (justify right bottom))
   )
+  (label "FLASH_CS" (at 93.98 128.27 180)
+    (effects (font (size 1.27 1.27)) (justify right bottom))
+  )
   (label "F0" (at 278.765 151.765 0)
     (effects (font (size 1.27 1.27)) (justify left bottom))
@@
     (effects (font (size 1.27 1.27)) (justify left bottom))
   )
-  (label "RGB_DATA" (at 114.3 128.27 180)
+  (label "RGB_DATA" (at 114.3 105.41 180)
     (effects (font (size 1.27 1.27)) (justify right bottom))
   )
@@
     (effects (font (size 1.27 1.27)) (justify left bottom))
   )
-  (label "FLASH_CS" (at 93.98 105.41 180)
-    (effects (font (size 1.27 1.27)) (justify right bottom))
-  )
   (label "B2" (at 113.665 238.125 0)
     (effects (font (size 1.27 1.27)) (justify left bottom))
@@
     (pin "2")
   )
-  (symbol (lib_id "power:+5V") (at 101.6 120.65 0) (unit 1)
+  (symbol (lib_id "power:+5V") (at 101.6 97.79 0) (unit 1)
     (in_bom yes) (on_board yes) (fields_autoplaced)
-    (property "Reference" "#PWR06" (id 0) (at 101.6 124.46 0)
+    (property "Reference" "#PWR06" (id 0) (at 101.6 101.6 0)
       (effects (font (size 1.27 1.27)) hide)
     )
-    (property "Value" "+5V" (id 1) (at 101.6 115.57 0))
-    (property "Footprint" "" (id 2) (at 101.6 120.65 0)
+    (property "Value" "+5V" (id 1) (at 101.6 92.71 0))
+    (property "Footprint" "" (id 2) (at 101.6 97.79 0)
       (effects (font (size 1.27 1.27)) hide)
     )
-    (property "Datasheet" "" (id 3) (at 101.6 120.65 0)
+    (property "Datasheet" "" (id 3) (at 101.6 97.79 0)
       (effects (font (size 1.27 1.27)) hide)
     )
@@
     (pin "3")
   )
-  (symbol (lib_id "keyboard-left-rescue:R-Device-keyboard-right-rescue") (at 101.6 124.46 180) (unit 1)
+  (symbol (lib_id "keyboard-left-rescue:R-Device-keyboard-right-rescue") (at 101.6 101.6 180) (unit 1)
     (in_bom yes) (on_board yes)
-    (property "Reference" "R5" (id 0) (at 104.14 124.46 90))
-    (property "Value" "5.1k" (id 1) (at 101.6 124.46 90))
-    (property "Footprint" "Resistor_SMD:R_0805_2012Metric_Pad1.20x1.40mm_HandSolder" (id 2) (at 103.378 124.46 90)
+    (property "Reference" "R5" (id 0) (at 104.14 101.6 90))
+    (property "Value" "5.1k" (id 1) (at 101.6 101.6 90))
+    (property "Footprint" "Resistor_SMD:R_0805_2012Metric_Pad1.20x1.40mm_HandSolder" (id 2) (at 103.378 101.6 90)
       (effects (font (size 1.27 1.27)) hide)
     )
-    (property "Datasheet" "~" (id 3) (at 101.6 124.46 0)
+    (property "Datasheet" "~" (id 3) (at 101.6 101.6 0)
       (effects (font (size 1.27 1.27)) hide)
     )
-    (property "Mouser" "C27834" (id 4) (at 101.6 124.46 0)
+    (property "Mouser" "C27834" (id 4) (at 101.6 101.6 0)
       (effects (font (size 1.27 1.27)) hide)
     )
-    (property "LCSC" "C104384" (id 5) (at 101.6 124.46 0)
+    (property "LCSC" "C104384" (id 5) (at 101.6 101.6 0)
       (effects (font (size 1.27 1.27)) hide)
     )

Commit message: Started rotating all switches; More progress on right half
Parts:
- removed T10, T11, T12, T16, T17, T18, T5, T6, T7, T9: TP, lakemountain:TestPoint_Pad_D1.0mm, symbol Connector:TestPoint
- removed U3: STM32F411CEU6, Bonsai_C4:QFN-48-1EP_7x7mm_P0.5mm_EP5.6x5.6mm_ThermalVias, symbol Bonsai_C4:STM32F411CEU6
- added S1: MX_stab, marbastlib-mx:STAB_MX_P_2.25u, symbol marbastlib-mx:MX_stab
- added SWcx1: MX_SW_HS, lakemountain:SW_MX_HS_1.75u_stp, symbol keyboard-mx:MX_SW_HS
- added SWdx1: MX_SW_HS, lakemountain:SW_MX_HS_2.25u, symbol keyboard-mx:MX_SW_HS
- added U3: STM32F411RETx, Package_QFP:LQFP-64_10x10mm_P0.5mm, symbol MCU_ST_STM32F4:STM32F411RETx
- LEDa1, LEDa2, LEDa3, LEDa4, LEDa5, LEDa6, LEDa7, LEDc2, LEDc3, LEDc4, LEDc5, LEDc6, LEDe1, LEDe2, LEDe3, LEDe4, LEDe5: footprint lakemountain:LED_MX_6028R_Flipped -> lakemountain:LED_MX_6028R
- LEDb1, LEDb2, LEDb3, LEDb4, LEDb5, LEDb6, LEDd3, LEDd4, LEDd5, LEDd6, LEDd7: footprint lakemountain:LED_MX_6028R -> lakemountain:LED_MX_6028R_Flipped
- LEDc1: footprint lakemountain:LED_MX_6028R_Flipped -> lakemountain:LED_MX_6028R_SOLO
- LEDd1, LEDd2: footprint lakemountain:LED_MX_6028R -> lakemountain:LED_MX_6028R_SOLO
- LS1: footprint Bonsai_C4:Buzzer_Mallory_AST1109MLTRQ -> lakemountain:Buzzer_Mallory_AST1109MLTRQ
- R12: footprint Resistor_SMD:R_0603_1608Metric -> Resistor_SMD:R_0805_2012Metric_Pad1.20x1.40mm_HandSolder
- R5: footprint Resistor_SMD:R_0805_2012Metric_Pad1.20x1.40mm_HandSolder -> Resistor_SMD:R_0603_1608Metric
- SWa1, SWa2, SWa3, SWa4, SWa5, SWa6, SWa7, SWb2, SWb3, SWb4, SWb5, SWb6, SWc2, SWc3, SWc4, SWc5, SWc6, SWd2, SWd3, SWd4, SWd5, SWd6, SWd7: footprint marbastlib-mx:SW_MX_HS_1u -> lakemountain:SW_MX_HS_1u
- SWb1: footprint marbastlib-mx:SW_MX_HS_1.5u -> lakemountain:SW_MX_HS_1.5u
- SWc1: footprint marbastlib-mx:SW_MX_HS_1.75u -> lakemountain:SW_MX_HS_1.75u
- SWd1, SWe1, SWe2, SWe3, SWe4: footprint marbastlib-mx:SW_MX_HS_1.25u -> lakemountain:SW_MX_HS_1.25u
- SWe6: footprint marbastlib-mx:SW_MX_HS_1.25u -> lakemountain:SW_MX_HS_2.25u
Connections:
- net +3.3V: now also R5.1, U3.1 (VBAT), U3.13 (VDDA), U3.19 (VDD), U3.32 (VDD), U3.48 (VDD), U3.64 (VDD); no longer R12.1
- net +5V: now also C7.1, R12.2; no longer C7.2, R5.2
- net B2: now also U3.28 (PB2); no longer SWa5.1, SWb5.1, SWc5.1, SWd5.1
- net BOOT0: now also U3.60 (BOOT0)
- net CONN_CS: now also U3.25 (PC5)
- net EEPROM_CS: now also U3.14 (PA0)
- net F0: now also U3.5 (PH0)
- net F1: now also U3.6 (PH1)
- net FLASH_CS: now also U3.24 (PC4)
- net GND: now also C7.2, U3.12 (VSSA), U3.18 (VSS), U3.31 (VSS), U3.47 (VSS), U3.63 (VSS); no longer C7.1
- net I2C1_SCL: now also R5.2, U3.61 (PB8); no longer R13.2
- net I2C1_SDA: now also R13.2, U3.62 (PB9); no longer R12.2
- net JTCK: now also U3.49 (PA14)
- net JTDI: now also U3.50 (PA15)
- net JTDO: now also U3.55 (PB3)
- net JTMS: now also U3.46 (PA13)
- net NRST: now also U3.7 (NRST)
- net RGB_DATA: now also R12.1, U3.15 (PA1); no longer R5.1
- net SPI_MISO: now also U3.56 (PB4)
- net SPI_MOSI: now also U3.57 (PB5)
- net SPLIT_HAND_PIN: now also U3.4 (PC15)
- net USART2_RX: now also U3.17 (PA3)
- net USART2_TX: now also U3.16 (PA2)
- net USB_D+: now also U3.45 (PA12)
- net USB_D-: now also U3.44 (PA11)
- net VBUS_DETECT: now also U3.42 (PA9)
- net VCAP_1: now also U3.30 (VCAP1)
- net audio1: now also U3.20 (PA4)
- net audio2: now also U3.21 (PA5)
- net col0: now also SWcx1.1, SWdx1.1, U3.59 (PB7)
- net col1: now also U3.58 (PB6)
- net col2: now also U3.26 (PB0)
- net col3: now also U3.27 (PB1)
- net col5: now also U3.33 (PB12)
- net col6: now also U3.34 (PB13)
- net row0: now also U3.35 (PB14)
- net row1: now also U3.36 (PB15)
- net row2: now also U3.22 (PA6)
- net row3: now also U3.23 (PA7)
- net row4: now also U3.41 (PA8)
- net at Dd1.2 (A), SWd1.2: now also SWdx1.2
- net at Dc1.2 (A), SWc1.2: now also SWcx1.2
- new net ENC_A: U3.52 (PC11)
- new net ENC_B: U3.53 (PC12)
- new net col4: SWa5.1, SWb5.1, SWc5.1, SWd5.1, U3.43 (PA10)
- no-connect marks 19 -> 30
Other:
- note added: "OBS: Left: TX on D-, RX on D+ Right: TX on D+, RX on D-"
- note removed: "Reset circuit from BonsaiC4 https://github.com/customMK/Bonsai-C"
- moved on the sheet: C7, T27

Commit message: Left PCB done, for now at least
Parts:
- removed D1: PMEG2010AEB, Bonsai_C4:D_SOD-523, symbol Bonsai_C4:PMEG2010AEB
- removed JP1, JP2: VBUS_SEL, Jumper:SolderJumper-3_P1.3mm_Open_RoundedPad1.0x1.5mm_NumberLabels, symbol Jumper:SolderJumper_3_Open
- added JP1: MUX_SEL, Jumper:SolderJumper-3_P1.3mm_Bridged12_RoundedPad1.0x1.5mm, symbol Jumper:SolderJumper_3_Bridged12
- added LOGO1: QMK Logo, lakemountain:QMK_PoweredBy, symbol Mechanical:Fiducial
- added LOGO2: OH Logo, Symbol:OSHW-Logo2_9.8x8mm_SilkScreen, symbol Mechanical:Fiducial
- added R15: 10k, Resistor_SMD:R_0603_1608Metric, symbol keyboard-left-rescue:R-Device-keyboard-right-rescue
- added U10, U11, U9: SRV05-4, Bonsai_C4:SOT-23-6, symbol Bonsai_C4:SRV05-4
- S1, S2, SWcx1, SWdx1: JLCPCB BOM (none) -> 0
Connections:
- net +3.3V: now also J3.A4 (VBUS), J3.A9 (VBUS), J3.B4 (VBUS), J3.B9 (VBUS), J6.A4 (VBUS), J6.A9 (VBUS), J6.B4 (VBUS), J6.B9 (VBUS), U10.5 (VP), U11.5 (VP)
- net CONN_CS: no longer J6.A8 (SBU1), J6.B8 (SBU2)
- net GND: now also R15.2, U10.2 (VN), U11.2 (VN), U9.2 (VN)
- net SPI_MISO: now also U11.6 (IO4)
- net USART2_RX: now also U9.3 (IO2)
- net USART2_TX: now also U9.1 (IO1)
- net USB_VBUS: now also U2.5 (VP)
- net USB_VBUS_IN_LINK: now also U9.5 (VP)
- net z1: now also U10.4 (IO3)
- net z2: now also U10.1 (IO1)
- net z3: now also U10.3 (IO2)
- net z4: now also U10.6 (IO4)
- net at J6.A6 (D+), J6.B6 (D+), JP4.2 (C): now also U11.1 (IO1)
- net at U1.11 (IN2), U1.21 (IN1): now also JP1.2 (C); no longer JP6.2 (C)
- net at J6.A7 (D-), J6.B7 (D-), JP3.2 (C): now also U11.3 (IO2)
- net CONN2_CS: now reaches U3.37 (PC6)
- net CONN2_CS: now also J6.A8 (SBU1), J6.B8 (SBU2), U11.4 (IO3)
- net CONN_SEL: now reaches U3.39 (PC8)
- net CONN_SEL: now also JP1.1 (A), R15.1
- net B2 renamed BOOT1
- net ENC_A: no longer names the net of U3.52 (PC11)
- net ENC_B: no longer names the net of U3.53 (PC12)
- new net: JP1.3 (B), JP6.2 (C)
- no-connect marks 30 -> 32
Other:
- note added: "Pull down CONN_SEL for default 0"
- note removed: "B2 is BOOT1"
- company: Lakemountain -> Lakemountain Keyboards
- moved on the sheet: FB4, H1, H2, H3, J4, J5, J6, JP3, JP4, JP6, JP7, JP8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

Commit message: Add all symbols and footprints to library
Parts:
- C1, C3: symbol Bonsai_C4:cap_1uF_10v_0402 -> lakemountain:cap_1uF_10v_0402
- C10, C11, C13, C14, C16, C17, C2: symbol Bonsai_C4:cap_100nF_16v_0402 -> lakemountain:cap_100nF_16v_0402
- C12, C18, C19, C20, C21, C22, C23, C6, C7: symbol Device:C -> lakemountain:C
- C15, C5: symbol Bonsai_C4:cap_4.7uF_10v_0402 -> lakemountain:cap_4.7uF_10v_0402
- C4: symbol Bonsai_C4:cap_10uF_10v_0402 -> lakemountain:cap_10uF_10v_0402
- C8, C9: symbol Bonsai_C4:cap_20pF_50v_0402 -> lakemountain:cap_20pF_50v_0402
- D3: symbol YAEMK:LED -> lakemountain:LED
- D4: symbol Bonsai_C4:SMD-LED-WHITE_0402_ -> lakemountain:SMD-LED-WHITE_0402_
- Da1, Da2, Da3, Da4, Da5, Da6, Da7, Db1, Db2, Db3, Db4, Db5, Db6, Dc1, Dc2, Dc3, Dc4, Dc5, Dc6, Dd1, Dd2, Dd3, Dd4, Dd5, Dd6, Dd7, De1, De2, De3, De4, De5, De6: symbol Device:D -> lakemountain:D
- F1, F2: symbol Bonsai_C4:SMD-PPTC-500MA_0805_ -> lakemountain:SMD-PPTC-500MA_0805_
- FB1, FB2, FB3, FB4: symbol Bonsai_C4:fb_0402_26ohm -> lakemountain:fb_0402_26ohm
- H1, H2, H3: symbol Mechanical:MountingHole_Pad -> lakemountain:MountingHole_Pad
- J1, J2, J3, J6: symbol keyboard-left-rescue:USB_C_Receptacle_USB2.0-Connector-keyboard-right-rescue -> lakemountain:USB_C_Receptacle_USB2.0-Connector-keyboard-right-rescue
- J4: symbol Connector_Generic:Conn_01x06 -> lakemountain:Conn_01x06
- J5: symbol marbastlib-various:JTAG_TC2030 -> lakemountain:JTAG_TC2030
- JP1: symbol Jumper:SolderJumper_3_Bridged12 -> lakemountain:SolderJumper_3_Bridged12
- JP3, JP4, JP6, JP7, JP8: symbol Jumper:SolderJumper_3_Open -> lakemountain:SolderJumper_3_Open
- LEDa1, LEDa2, LEDa3, LEDa4, LEDa5, LEDa6, LEDa7, LEDb1, LEDb2, LEDb3, LEDb4, LEDb5, LEDb6, LEDc1, LEDc2, LEDc3, LEDc4, LEDc5, LEDc6, LEDd1, LEDd2, LEDd3, LEDd4, LEDd5, LEDd6, LEDd7, LEDe1, LEDe2, LEDe3, LEDe4, LEDe5, LEDs1, LEDs10, LEDs11, LEDs12, LEDs13, LEDs14, LEDs15, LEDs16, LEDs17, LEDs2, LEDs3, LEDs4, LEDs5, LEDs6, LEDs7, LEDs8, LEDs9: symbol keyboard-mx:MX_SK6812MINI-E -> lakemountain:MX_SK6812MINI-E
- LOGO1, LOGO2: symbol Mechanical:Fiducial -> lakemountain:Fiducial
- LS1: symbol keyboard-left-rescue:Speaker-Device-keyboard-right-rescue -> lakemountain:Speaker-Device-keyboard-right-rescue
- Q1, Q3: symbol Bonsai_C4:MUN5311DW1T1G -> lakemountain:MUN5311DW1T1G
- Q2: symbol Transistor_FET:AO3401A -> lakemountain:AO3401A
- R1, R11, R12, R13, R15, R2, R3, R5: symbol keyboard-left-rescue:R-Device-keyboard-right-rescue -> lakemountain:R-Device-keyboard-right-rescue
- R10: symbol Bonsai_C4:r_470_0402_1p -> lakemountain:r_470_0402_1p
- R14, R6: symbol Bonsai_C4:r_75_0402_1p -> lakemountain:r_75_0402_1p
- R4: symbol keyboard-left-rescue:R-Device-keyboard-right-rescue -> lakemountain:R-Device-keyboard-right-rescue; now not fitted
- R7: symbol Bonsai_C4:r_4.7k_0402_1p -> lakemountain:r_4.7k_0402_1p
- R8: symbol Bonsai_C4:r_10k_0402_1p -> lakemountain:r_10k_0402_1p
- R9: symbol Bonsai_C4:r_100k_0402_1p -> lakemountain:r_100k_0402_1p
- S1: footprint marbastlib-mx:STAB_MX_P_2.25u -> lakemountain:STAB_MX_P_2.25u; symbol marbastlib-mx:MX_stab -> lakemountain:MX_stab; now not fitted
- S2: footprint marbastlib-mx:STAB_MX_P_2.25u -> lakemountain:STAB_MX_P_2.25u; symbol marbastlib-mx:MX_stab -> lakemountain:MX_stab
- SW1: symbol keyboard_parts:SW_PUSH -> lakemountain:SW_PUSH
- SWa1, SWa2, SWa3, SWa4, SWa5, SWa6, SWa7, SWb1, SWb2, SWb3, SWb4, SWb5, SWb6, SWc1, SWc2, SWc3, SWc4, SWc5, SWc6, SWd1, SWd2, SWd3, SWd4, SWd5, SWd6, SWd7, SWe1, SWe2, SWe3, SWe4, SWe6: symbol keyboard-mx:MX_SW_HS -> lakemountain:MX_SW_HS
- SWcx1, SWdx1: symbol keyboard-mx:MX_SW_HS -> lakemountain:MX_SW_HS; now not fitted
- T1, T13, T14, T15, T19, T2, T20, T21, T22, T23, T24, T25, T26, T27, T3, T4, T8: symbol Connector:TestPoint -> lakemountain:TestPoint
- U1: symbol Analog_Switch:TS3A27518ERTW -> lakemountain:TS3A27518ERTW
- U10, U11, U2, U9: symbol Bonsai_C4:SRV05-4 -> lakemountain:SRV05-4
- U3: symbol MCU_ST_STM32F4:STM32F411RETx -> lakemountain:STM32F411RETx
- U4: symbol Bonsai_C4:MB85RS64PNF-G-JNERE1 -> lakemountain:MB85RS64PNF-G-JNERE1
- U5: symbol Bonsai_C4:AAP2967-33VIR1 -> lakemountain:AAP2967-33VIR1
- U6: symbol Amplifier_Operational:LMV321 -> lakemountain:LMV321
- U7: symbol Bonsai_C4:W25Q128JVSIQ -> lakemountain:W25Q128JVSIQ
- U8: symbol Bonsai_C4:SN74LV1T34DCKR -> lakemountain:SN74LV1T34DCKR
- Y1: symbol Bonsai_C4:SMD-CRYSTAL-8MHZ-20PF-10PPM_2P-5.0X3.2MM_ -> lakemountain:SMD-CRYSTAL-8MHZ-20PF-10PPM_2P-5.0X3.2MM_
Other:
- moved on the sheet: J4, J5, U4, U7

Commit message: Remove unused libs
Parts:
- C1, C10, C11, C13, C14, C15, C16, C17, C2, C3, C4, C5, C8, C9: footprint Bonsai_C4:C_0402_1005Metric -> lakemountain:C_0402_1005Metric
- C12, C18, C19, C20, C21, C22, C23, C6, C7: footprint Bonsai_C4:C_0805 -> lakemountain:C_0805
- D3: footprint LED_SMD:LED_0603_1608Metric -> lakemountain:LED_0603_1608Metric
- D4: footprint Bonsai_C4:LED_0402 -> lakemountain:LED_0402
- Da1, Da2, Da3, Da4, Da5, Da6, Da7, Db1, Db2, Db3, Db4, Db5, Db6, Dc1, Dc2, Dc3, Dc4, Dc5, Dc6, Dd1, Dd2, Dd3, Dd4, Dd5, Dd6, Dd7, De1, De2, De3, De4, De6: footprint Diode_SMD:D_SOD-123 -> lakemountain:D_SOD-123
- De5: footprint Bonsai_C4:D_SOD-523 -> lakemountain:D_SOD-523
- F1, F2: footprint Bonsai_C4:F1206 -> lakemountain:F1206
- FB1, FB2, FB3, FB4, R10, R14, R6, R7, R8, R9: footprint Bonsai_C4:R_0402_1005Metric -> lakemountain:R_0402_1005Metric
- H1, H2, H3: footprint MountingHole:MountingHole_2.2mm_M2_Pad_Via -> lakemountain:MountingHole_2.2mm_M2_Pad_Via
- J4: footprint Connector_PinHeader_2.54mm:PinHeader_1x06_P2.54mm_Vertical -> lakemountain:PinHeader_1x06_P2.54mm_Vertical
- J5: footprint marbastlib-various:CON_TC2030_outlined -> lakemountain:CON_TC2030_outlined
- JP1: footprint Jumper:SolderJumper-3_P1.3mm_Bridged12_RoundedPad1.0x1.5mm -> lakemountain:SolderJumper-3_P1.3mm_Bridged12_RoundedPad1.0x1.5mm
- JP3, JP4, JP6, JP7, JP8: footprint Jumper:SolderJumper-3_P1.3mm_Open_RoundedPad1.0x1.5mm_NumberLabels -> lakemountain:SolderJumper-3_P1.3mm_Open_RoundedPad1.0x1.5mm_NumberLabels
- LOGO2: footprint Symbol:OSHW-Logo2_9.8x8mm_SilkScreen -> lakemountain:OSHW-Logo2_9.8x8mm_SilkScreen
- Q1, Q3: footprint Bonsai_C4:SOT-363_SC-70-6_SC-88 -> lakemountain:SOT-363_SC-70-6_SC-88
- Q2: footprint Package_TO_SOT_SMD:SOT-23 -> lakemountain:SOT-23
- R1, R11, R13, R15, R2, R3, R4, R5: footprint Resistor_SMD:R_0603_1608Metric -> lakemountain:R_0603_1608Metric
- R12: footprint Resistor_SMD:R_0805_2012Metric_Pad1.20x1.40mm_HandSolder -> lakemountain:R_0805_2012Metric_Pad1.20x1.40mm_HandSolder
- SW1: footprint Button_Switch_SMD:SW_SPST_TL3342 -> lakemountain:SW_SPST_TL3342
- U1: footprint Package_DFN_QFN:WQFN-24-1EP_4x4mm_P0.5mm_EP2.6x2.6mm -> lakemountain:WQFN-24-1EP_4x4mm_P0.5mm_EP2.6x2.6mm
- U10, U11, U2, U9: footprint Bonsai_C4:SOT-23-6 -> lakemountain:SOT-23-6
- U3: footprint Package_QFP:LQFP-64_10x10mm_P0.5mm -> lakemountain:LQFP-64_10x10mm_P0.5mm
- U4: footprint Bonsai_C4:SOP-8_3.9x4.9mm_P1.27mm -> lakemountain:SOP-8_3.9x4.9mm_P1.27mm
- U5: footprint Bonsai_C4:SOT-23-5 -> lakemountain:SOT-23-5
- U6: footprint Package_TO_SOT_SMD:SOT-23-5 -> lakemountain:SOT-23-5
- U7: footprint Bonsai_C4:SOIC-8_5.23x5.23mm_P1.27mm -> lakemountain:SOIC-8_5.23x5.23mm_P1.27mm
- U8: footprint Bonsai_C4:SOT-353_SC-70-5 -> lakemountain:SOT-353_SC-70-5
- Y1: footprint Bonsai_C4:X2-SMD-5.0X3.2X1.3MM -> lakemountain:X2-SMD-5.0X3.2X1.3MM

Commit message: Right PCB routed. Needs DRC and some symbol fixing.
Parts:
- added JP2: SPI/I2C, Jumper:SolderJumper-3_P1.3mm_Open_RoundedPad1.0x1.5mm_NumberLabels, symbol Jumper:SolderJumper_3_Open
- added JP5, JP9: 5V/3V3, lakemountain:SolderJumper-3_P1.3mm_Bridged12_RoundedPad1.0x1.5mm, symbol lakemountain:SolderJumper_3_Bridged12
- LEDs1, LEDs10, LEDs11, LEDs12, LEDs13, LEDs14, LEDs15, LEDs16, LEDs17, LEDs2, LEDs3, LEDs4, LEDs5, LEDs6, LEDs7, LEDs8, LEDs9: value MX_SK6812MINI-E -> sk6812side
Connections:
- net +3.3V: now also J4.6 (Pin_6), JP5.3 (B), JP9.3 (B); no longer J3.A4 (VBUS), J3.A9 (VBUS), J3.B4 (VBUS), J3.B9 (VBUS), J4.1 (Pin_1), J6.A4 (VBUS), J6.A9 (VBUS), J6.B4 (VBUS), J6.B9 (VBUS), U10.5 (VP), U11.5 (VP)
- net +5V: now also JP5.1 (A), JP9.1 (A)
- net GND: now also J4.1 (Pin_1); no longer J4.6 (Pin_6)
- net JTCK: now also J4.3 (Pin_3); no longer J4.4 (Pin_4)
- net JTDI: now also J4.5 (Pin_5); no longer J4.2 (Pin_2)
- net JTDO: now also J4.4 (Pin_4); no longer J4.3 (Pin_3)
- net JTMS: now also J4.2 (Pin_2); no longer J4.5 (Pin_5)
- net SPI_MISO: now also JP2.1 (A); no longer U1.23 (NC1)
- net JOY_X: now reaches U3.38 (PC7)
- net JOY_X: now also JP2.3 (B)
- new net: J6.A4 (VBUS), J6.A9 (VBUS), J6.B4 (VBUS), J6.B9 (VBUS), JP9.2 (C), U11.5 (VP)
- new net: J3.A4 (VBUS), J3.A9 (VBUS), J3.B4 (VBUS), J3.B9 (VBUS), JP5.2 (C), U10.5 (VP)
- new net x1: JP2.2 (C), U1.23 (NC1)
- no-connect marks 32 -> 31
