File: Left/left.kicad_pcb (KiCad board)
At the start: 2 copper layers, 135.6 x 112.3 mm, 214 parts, among them J1 USB_EXT, J2 USB_Conn_1, J3 USB_Link, J4 Conn_01x06, J5 JTAG_TC2030, J6 USB_Conn_2, Q1 MUN5311DW1T1G, Q2 AO3401A, Q3 MUN5311DW1T1G, SW1 Reset, T1 TP, T13 TP, T14 TP, T15 TP, T19 TP, T2 TP, T20 TP, T21 TP, T22 TP, T23 TP, T24 3V3, T25 5V, T26 GND, T27 GND, T3 TP, T4 TP, T8 TP, U1 TS3A27518ERTW, U10 SRV05-4, U11 SRV05-4, U2 SRV05-4, U3 STM32F411RETx, U4 MB85RS64PNF-G-JNERE1, U5 AAP2967-33VIR1, U6 LMV321, U7 W25Q128JVSIQ, U8 SN74LV1T34DCKR, U9 SRV05-4, Y1 SMD-CRYSTAL-8MHZ-20PF-10PPM_2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

Commit message: Right PCB routed. Needs DRC and some symbol fixing.
Parts:
- added JP2: SPI/I2C, Jumper:SolderJumper-3_P1.3mm_Open_RoundedPad1.0x1.5mm_NumberLabels, B.Cu at (158.2, 59.7)
- added JP5: 5V/3V3, lakemountain:SolderJumper-3_P1.3mm_Bridged12_RoundedPad1.0x1.5mm, B.Cu at (186.7, 144.7)
- added JP9: 5V/3V3, lakemountain:SolderJumper-3_P1.3mm_Bridged12_RoundedPad1.0x1.5mm, B.Cu at (180.6, 54.7)
- LEDs1, LEDs10, LEDs11, LEDs12, LEDs13, LEDs14, LEDs15, LEDs16, LEDs17, LEDs2, LEDs3, LEDs4, LEDs5, LEDs6, LEDs7, LEDs8, LEDs9: value MX_SK6812MINI-E -> sk6812side
- moved C6 77.4 mm to (94.1, 73.0), turned to -90 degrees
- moved J4 12.7 mm to (65.7, 84.5), turned to 0 degrees
Connections:
- J3 pad A4: +3.3V -> Net-(JP5-C)
- J3 pad A9: +3.3V -> Net-(JP5-C)
- J3 pad B4: +3.3V -> Net-(JP5-C)
- J3 pad B9: +3.3V -> Net-(JP5-C)
- J4 pad 1: +3.3V -> GND
- J4 pad 2: JTDI -> JTMS
- J4 pad 3: JTDO -> JTCK
- J4 pad 4: JTCK -> JTDO
- J4 pad 5: JTMS -> JTDI
- J4 pad 6: GND -> +3.3V
- J6 pad A4: +3.3V -> Net-(JP9-C)
- J6 pad A9: +3.3V -> Net-(JP9-C)
- J6 pad B4: +3.3V -> Net-(JP9-C)
- J6 pad B9: +3.3V -> Net-(JP9-C)
- U1 pad 23: /SPI_MISO -> /x1
- U10 pad 5: +3.3V -> Net-(JP5-C)
- U11 pad 5: +3.3V -> Net-(JP9-C)
- U3 pad 38: unconnected-(U3-PC7-Pad38) -> /JOY_X
Routing:
- net /x1: track 0.00 -> 97.3 mm, vias 0 -> 4
- net /SPI_MISO: track 233.7 -> 143.4 mm, vias 14 -> 11
- net /JOY_X: track 0.00 -> 88.3 mm, vias 0 -> 4
- net +3.3V: track 608.4 -> 569.6 mm, vias 41 -> 35
- net Net-(JP5-C): track 0.00 -> 24.5 mm, vias 0 -> 2
- net Net-(JP9-C): track 0.00 -> 23.7 mm, vias 0 -> 5
- net +5V: track 923.7 -> 945.4 mm, vias 45 -> 48
- net GND: track 165.9 -> 169.3 mm, vias 209 -> 215
- net /col1: track 130.3 -> 131.5 mm, vias 5 -> 6
- net /CONN_SEL: track 153.5 -> 154.1 mm

Commit message: Push latest, don't remember changes...
Parts:
- removed the G*** at (152.1, 44.4)
