File: right/right.kicad_sch (KiCad schematic)
At the start: 250 parts, among them J1 USB_EXT, J2 Conn_01x06, J3 USB_Conn_1, J4 JTAG_TC2030, J5 USB_Link, J6 USB_Conn_2, Q1 MUN5311DW1T1G, Q2 MUN5311DW1T1G, Q3 AO3401A, SW1 Reset, T1 TP, T10 TP, T11 TP, T12 TP, T13 TP, T14 TP, T15 TP, T16 TP, T17 TP, T18 TP, T19 TP, T2 TP, T20 TP, T21 TP, T22 TP, T23 TP, T24 3V3, T25 5V, T26 GND, T27 GND, T3 TP, T4 TP, T5 TP, T6 TP, T7 TP, T8 TP, T9 TP, U1 STM32F411RETx, U2 AAP2967-33VIR1, U4 SRV05-4, U5 SN74LV1T34DCKR, U6 LMV321, U7 MB85RS64PNF-G-JNERE1, U8 W25Q128JVSIQ, U9 TS3A27518ERTW, Y1 SMD-CRYSTAL-8MHZ-20PF-10PPM_2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

Commit message: Before rotating switches and LEDs...
Parts:
- added C24, C25, C26, C27, C28, C29, C30, C31: 100n, Bonsai_C4:C_0805, symbol Device:C
Connections:
- net +5V: now also C24.1, C25.2, C26.1, C27.2, C28.1, C29.1, C30.2, C31.1
- net FLASH_CS: now also U1.43 (PA10); no longer U1.15 (PA1)
- net GND: now also C24.2, C25.1, C26.2, C27.1, C28.2, C29.2, C30.1, C31.2
- net RGB_DATA: now also U1.15 (PA1); no longer U1.43 (PA10)
Other:
- moved on the sheet: C13, C14, C15, C16, C17, C18, C19, C20, C21, JP10, JP8, JP9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

Commit message: Started rotating all switches; More progress on right half
Parts:
- added JP?: SPI/I2C, Jumper:SolderJumper-3_P1.3mm_Open_RoundedPad1.0x1.5mm_NumberLabels, symbol Jumper:SolderJumper_3_Open
- added S4: MX_stab, lakemountain:STAB_MX_P_2.25u, symbol marbastlib-mx:MX_stab
- added SWbx8: MX_SW_HS, lakemountain:SW_MX_HS_1.5u, symbol keyboard-mx:MX_SW_HS
- added SWcx7: MX_SW_HS, lakemountain:SW_MX_HS_2.25u, symbol keyboard-mx:MX_SW_HS
- added SWe10, SWe11, SWe8, SWe9: MX_SW_HS, lakemountain:SW_MX_HS_1.25u, symbol keyboard-mx:MX_SW_HS
- LEDa1, LEDa2, LEDa3, LEDa4, LEDa5, LEDa6, LEDa7, LEDa8, LEDc1, LEDc2, LEDc3, LEDc4, LEDc5, LEDc6, LEDc8, LEDe1, LEDe2, LEDe3, LEDe4, LEDe5, LEDe6, LEDe7: footprint lakemountain:LED_MX_6028R_Flipped -> lakemountain:LED_MX_6028R
- LEDb1, LEDb2, LEDb3, LEDb4, LEDb5, LEDb6, LEDb7, LEDb8, LEDb9, LEDd1, LEDd2, LEDd3, LEDd4, LEDd5, LEDd6, LEDd7, LEDd8: footprint lakemountain:LED_MX_6028R -> lakemountain:LED_MX_6028R_Flipped
- LEDc7: footprint lakemountain:LED_MX_6028R_Flipped -> lakemountain:LED_MX_6028R_SOLO
- SWa7: footprint lakemountain:SW_MX_HS_1.75u -> lakemountain:SW_MX_HS_2u
Connections:
- net B2: now also SWe9.2
- net SPI_MISO: now also JP?.1 (A); no longer U9.23 (NC1)
- net USART2_RX: now also J3.A7 (D-), J3.B7 (D-); no longer J3.A6 (D+), J3.B6 (D+)
- net USART2_TX: now also J3.A6 (D+), J3.B6 (D+); no longer J3.A7 (D-), J3.B7 (D-)
- net col1: no longer SWe1.1
- net col2: now also SWe1.1
- net col3: now also SWe8.1
- net col5: now also SWe10.2
- net col6: now also SWcx7.2
- net col7: now also SWbx8.1, SWe11.1
- net at Db9.2 (A), SWe5.2: now also SWe10.1
- net at Db8.2 (A), SWc7.2: now also SWcx7.1
- net at De4.2 (A), SWe4.2: now also SWe9.1
- net at De3.2 (A), SWe2.2: now also SWe8.2
- net at De5.2 (A), SWe6.2: now also SWe11.2
- net at Db10.2 (A), SWb8.2: now also SWbx8.2
- net JOY_X: now reaches U1.2 (PC13)
- net JOY_X: now also JP?.3 (B)
- new net x1: JP?.2 (C), U9.23 (NC1)
- no-connect marks 31 -> 30
Other:
- note added: "OBS: Left: TX on D-, RX on D+ Right: TX on D+, RX on D-"
- moved on the sheet: De2, JP6, JP7, SWe1

Commit message: Left PCB done, for now at least
Parts:
- added S5: MX_stab, lakemountain:STAB_MX_P_2.25u, symbol marbastlib-mx:MX_stab
- added SWd9: MX_SW_HS, lakemountain:SW_MX_HS_2.75u, symbol keyboard-mx:MX_SW_HS
- LEDd6: footprint lakemountain:LED_MX_6028R_Flipped -> lakemountain:LED_MX_6028R_SOLO
- gave numbers to parts that had none: 1
Connections:
- net col0: now also U9.8 (NO1)
- net col6: now also SWd9.2; no longer U9.8 (NO1)
- net row0: now also U9.10 (NO2)
- net row1: no longer U9.10 (NO2)
- net row2: no longer U9.12 (NO3)
- net row3: now also U9.12 (NO3)
- net at Dd6.2 (A), SWd6.2: now also SWd9.1
- net ENC_2_A: now reaches U1.40 (PC9)
- net ENC_2_B: now reaches U1.51 (PC10)
- no-connect marks 30 -> 28
Changed lines of the file:
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@@
   (junction (at 176.53 130.81) (diameter 0) (color 0 0 0 0)
   )
+  (junction (at 227.33 135.89) (diameter 0) (color 0 0 0 0)
+  )
   (junction (at 144.78 375.92) (diameter 0) (color 0 0 0 0)
   )
@@
   (no_connect (at 46.99 104.14))
   (no_connect (at 46.99 109.22))
-  (no_connect (at 46.99 129.54))
   (no_connect (at 57.15 374.65))
   (no_connect (at 434.34 266.7))
@@
   (no_connect (at 46.99 124.46))
   (no_connect (at 46.99 121.92))
-  (no_connect (at 46.99 127))
   (no_connect (at 312.42 237.49))
   (no_connect (at 312.42 234.95))
@@
     (stroke (width 0) (type default) (color 0 0 0 0))
   )
+  (wire (pts (xy 39.37 134.62) (xy 46.99 134.62))
+    (stroke (width 0) (type default) (color 0 0 0 0))
+  )
   (wire (pts (xy 473.71 314.96) (xy 473.71 316.23))
     (stroke (width 0) (type default) (color 0 0 0 0))
@@
     (stroke (width 0) (type default) (color 0 0 0 0))
   )
+  (wire (pts (xy 39.37 132.08) (xy 46.99 132.08))
+    (stroke (width 0) (type default) (color 0 0 0 0))
+  )
   (wire (pts (xy 544.83 292.1) (xy 549.91 292.1))
     (stroke (width 0) (type default) (color 0 0 0 0))
@@
     (stroke (width 0) (type default) (color 0 0 0 0))
   )
+  (wire (pts (xy 227.33 135.89) (xy 232.41 135.89))
+    (stroke (width 0) (type default) (color 0 0 0 0))
+  )
   (wire (pts (xy 246.38 90.17) (xy 246.38 110.49))
     (stroke (width 0) (type default) (color 0 0 0 0))
   )
+  (wire (pts (xy 36.83 127) (xy 46.99 127))
+    (stroke (width 0) (type default) (color 0 0 0 0))
+  )
   (wire (pts (xy 407.67 73.66) (xy 422.91 73.66))
     (stroke (width 0) (type default) (color 0 0 0 0))
@@
     (stroke (width 0) (type default) (color 0 0 0 0))
   )
+  (wire (pts (xy 36.83 129.54) (xy 46.99 129.54))
+    (stroke (width 0) (type default) (color 0 0 0 0))
+  )
   (wire (pts (xy 659.13 134.62) (xy 659.13 121.92))
     (stroke (width 0) (type default) (color 0 0 0 0))
@@
     (stroke (width 0) (type default) (color 0 0 0 0))
   )
-  (wire (pts (xy 39.37 132.08) (xy 46.99 132.08))
-    (stroke (width 0) (type default) (color 0 0 0 0))
-  )
   (wire (pts (xy 556.26 264.16) (xy 544.83 264.16))
     (stroke (width 0) (type default) (color 0 0 0 0))
@@
     (stroke (width 0) (type default) (color 0 0 0 0))
   )
+  (wire (pts (xy 222.25 130.81) (xy 227.33 130.81))
+    (stroke (width 0) (type default) (color 0 0 0 0))
+  )
   (wire (pts (xy 53.34 189.865) (xy 63.5 189.865))
     (stroke (width 0) (type default) (color 0 0 0 0))
@@
     (stroke (width 0) (type default) (color 0 0 0 0))
   )
-  (wire (pts (xy 39.37 134.62) (xy 46.99 134.62))
-    (stroke (width 0) (type default) (color 0 0 0 0))
-  )
   (polyline (pts (xy 16.51 203.2) (xy 201.93 203.2))
     (stroke (width 0) (type default) (color 0 0 0 0))
@@
     (effects (font (size 1.27 1.27)) (justify left bottom))
   )
-  (label "ENC_B" (at 39.37 134.62 0)
-    (effects (font (size 1.27 1.27)) (justify left bottom))
-  )
   (label "USART2_TX" (at 313.69 367.03 180)
     (effects (font (size 1.27 1.27)) (justify right bottom))
@@
     (effects (font (size 1.27 1.27)) (justify right bottom))
   )
-  (label "col6" (at 440.69 254 180)
+  (label "col0" (at 440.69 254 180)
     (effects (font (size 1.27 1.27)) (justify right bottom))
   )
@@
     (effects (font (size 1.27 1.27)) (justify right bottom))
   )
+  (label "ENC_2_B" (at 36.83 129.54 0)
+    (effects (font (size 1.27 1.27)) (justify left bottom))
+  )
   (label "x1" (at 434.34 236.22 0)
     (effects (font (size 1.27 1.27)) (justify left bottom))
   )
+  (label "ENC_A" (at 39.37 132.08 0)
+    (effects (font (size 1.27 1.27)) (justify left bottom))
+  )
   (label "col5" (at 210.82 179.07 90)
     (effects (font (size 1.27 1.27)) (justify left bottom))
@@
     (effects (font (size 1.27 1.27)) (justify right bottom))
   )
-  (label "row1" (at 440.69 256.54 180)
+  (label "row0" (at 440.69 256.54 180)
     (effects (font (size 1.27 1.27)) (justify right bottom))
   )
@@
     (effects (font (size 1.27 1.27)) (justify right bottom))
   )
-  (label "ENC_A" (at 39.37 132.08 0)
-    (effects (font (size 1.27 1.27)) (justify left bottom))
-  )
   (label "USB_VBUS" (at 556.26 279.4 180)
     (effects (font (size 1.27 1.27)) (justify right bottom))
@@
     (effects (font (size 1.27 1.27)) (justify left bottom))
   )
+  (label "ENC_B" (at 39.37 134.62 0)
+    (effects (font (size 1.27 1.27)) (justify left bottom))
+  )
   (label "USB_D-" (at 91.44 91.44 180)
     (effects (font (size 1.27 1.27)) (justify right bottom))
@@
     (effects (font (size 1.27 1.27)) (justify left bottom))
   )
-  (label "row2" (at 440.69 259.08 180)
+  (label "row3" (at 440.69 259.08 180)
     (effects (font (size 1.27 1.27)) (justify right bottom))
   )
@@
     (effects (font (size 1.27 1.27)) (justify left bottom))
   )
+  (label "ENC_2_A" (at 36.83 127 0)
+    (effects (font (size 1.27 1.27)) (justify left bottom))
+  )
   (label "I2C1_SDA" (at 92.71 129.54 180)
     (effects (font (size 1.27 1.27)) (justify right bottom))
@@
     (pin "1")
   )
+  (symbol (lib_id "keyboard-mx:MX_SW_HS") (at 229.87 133.35 180) (unit 1)
+    (in_bom yes) (on_board yes) (fields_autoplaced)
+    (property "Reference" "SWd9" (id 0) (at 229.87 125.73 0))
+    (property "Value" "MX_SW_HS" (id 1) (at 229.87 128.27 0))
+    (property "Footprint" "lakemountain:SW_MX_HS_2.75u" (id 2) (at 229.87 133.35 0)
+      (effects (font (size 1.27 1.27)) hide)
+    )
+    (property "Datasheet" "~" (id 3) (at 229.87 133.35 0)
+      (effects (font (size 1.27 1.27)) hide)
+    )
+    (property "LCSC" "C2803348" (id 4) (at 229.87 133.35 0)
+      (effects (font (size 1.27 1.27)) hide)
+    )
+    (pin "1")
+    (pin "2")
+  )
   (symbol (lib_id "keyboard-mx:MX_SK6812MINI-E") (at 438.15 81.28 0) (unit 1)
     (in_bom yes) (on_board yes)
@@
       (effects (font (size 1.27 1.27)) hide)
     )
-    (property "Footprint" "lakemountain:LED_MX_6028R_Flipped" (id 2) (at 468.63 127 0)
+    (property "Footprint" "lakemountain:LED_MX_6028R_SOLO" (id 2) (at 468.63 127 0)
       (effects (font (size 1.27 1.27)) hide)
     )
@@
     (pin "2")
   )
+  (symbol (lib_id "marbastlib-mx:MX_stab") (at 266.7 135.89 0) (unit 1)
+    (in_bom yes) (on_board yes) (fields_autoplaced)
+    (property "Reference" "S5" (id 0) (at 273.05 134.4929 0)
+      (effects (font (size 1.27 1.27)) (justify left))
+    )
+    (property "Value" "MX_stab" (id 1) (at 273.05 137.0329 0)
+      (effects (font (size 1.27 1.27)) (justify left))
+    )
+    (property "Footprint" "lakemountain:STAB_MX_P_2.25u" (id 2) (at 266.7 135.89 0)
+      (effects (font (size 1.27 1.27)) hide)
+    )
+    (property "Datasheet" "" (id 3) (at 266.7 135.89 0)
+      (effects (font (size 1.27 1.27)) hide)
+    )
+  )
   (symbol (lib_id "Connector:TestPoint") (at 544.83 276.86 90) (unit 1)
     (in_bom yes) (on_board yes) (fields_autoplaced)
@@
   (symbol (lib_id "Jumper:SolderJumper_3_Open") (at 427.99 278.13 270) (unit 1)
     (in_bom yes) (on_board yes) (fields_autoplaced)
-    (property "Reference" "JP?" (id 0) (at 430.53 276.8599 90)
+    (property "Reference" "JP11" (id 0) (at 430.53 276.8599 90)
       (effects (font (size 1.27 1.27)) (justify left))
     )
@@
     )
     (path "/bd68a45f-2f2b-48c8-bcd0-333be48c66d2"
-      (reference "JP?") (unit 1) (value "SPI/I2C") (footprint "Jumper:SolderJumper-3_P1.3mm_Open_RoundedPad1.0x1.5mm_NumberLabels")
+      (reference "JP11") (unit 1) (value "SPI/I2C") (footprint "Jumper:SolderJumper-3_P1.3mm_Open_RoundedPad1.0x1.5mm_NumberLabels")
     )
     (path "/2060ef9a-5f73-4b22-b2fd-99c6e6599e0d"
@@
     )
     (path "/34aef76a-977a-45dc-a411-d20ca33846c9"
-      (reference "LEDd6") (unit 1) (value "MX_SK6812MINI-E") (footprint "lakemountain:LED_MX_6028R_Flipped")
+      (reference "LEDd6") (unit 1) (value "MX_SK6812MINI-E") (footprint "lakemountain:LED_MX_6028R_SOLO")
     )
     (path "/6197f5ce-0845-443d-bb03-fb6f4b8b4b8c"
@@
       (reference "S4") (unit 1) (value "MX_stab") (footprint "lakemountain:STAB_MX_P_2.25u")
     )
+    (path "/5cabde4e-287d-4568-b2e7-d3ea51f3ad3f"
+      (reference "S5") (unit 1) (value "MX_stab") (footprint "lakemountain:STAB_MX_P_2.25u")
+    )
     (path "/889d8555-4687-45dd-a753-ca74d5ce8f4d"
       (reference "SW1") (unit 1) (value "Reset") (footprint "Button_Switch_SMD:SW_SPST_TL3342")
@@
       (reference "SWd8") (unit 1) (value "MX_SW_HS") (footprint "lakemountain:SW_MX_HS_1u")
     )
+    (path "/04b451a5-3230-4293-b006-0bb49a785059"
+      (reference "SWd9") (unit 1) (value "MX_SW_HS") (footprint "lakemountain:SW_MX_HS_2.75u")
+    )
     (path "/c062b6ef-88f2-4bf9-baa0-622b051c8bee"

Commit message: Right PCB routed. Needs DRC and some symbol fixing.
Parts:
- removed JP1, JP2: VBUS_SEL, Jumper:SolderJumper-3_P1.3mm_Open_RoundedPad1.0x1.5mm_NumberLabels, symbol Jumper:SolderJumper_3_Open
- removed JP10, JP8, JP9: SolderJumper_2_Open, Jumper:SolderJumper-2_P1.3mm_Open_RoundedPad1.0x1.5mm, symbol Jumper:SolderJumper_2_Open
- removed JP11, JP6, JP7: SPI/I2C, Jumper:SolderJumper-3_P1.3mm_Open_RoundedPad1.0x1.5mm_NumberLabels, symbol Jumper:SolderJumper_3_Open
- removed JP5: MUX_SEL, Jumper:SolderJumper-3_P1.3mm_Open_RoundedPad1.0x1.5mm_NumberLabels, symbol Jumper:SolderJumper_3_Open
- removed T1, T10, T11, T12, T13, T14, T15, T16, T17, T18, T19, T2, T20, T21, T22, T23, T3, T4, T5, T6, T7, T8, T9: TP, lakemountain:TestPoint_Pad_D1.0mm, symbol Connector:TestPoint
- removed T24: 3V3, lakemountain:TestPoint_Pad_D1.0mm, symbol Connector:TestPoint
- removed T25: 5V, lakemountain:TestPoint_Pad_D1.0mm, symbol Connector:TestPoint
- removed T26, T27: GND, lakemountain:TestPoint_Pad_D1.0mm, symbol Connector:TestPoint
- added JP1: 60%, Jumper:SolderJumper-2_P1.3mm_Open_RoundedPad1.0x1.5mm, symbol lakemountain:SolderJumper_2_Open
- added JP1: MUX_SEL, lakemountain:SolderJumper-3_P1.3mm_Bridged12_RoundedPad1.0x1.5mm, symbol lakemountain:SolderJumper_3_Bridged12
- added JP2: SolderJumper_3_Bridged12, Jumper:SolderJumper-3_P1.3mm_Bridged2Bar12_RoundedPad1.0x1.5mm, symbol lakemountain:SolderJumper_3_Bridged12
- added JP6: MUX_SEL, lakemountain:SolderJumper-3_P1.3mm_Open_RoundedPad1.0x1.5mm_NumberLabels, symbol lakemountain:SolderJumper_3_Open
- added JP8: Jumper:SolderJumper-3_P1.3mm_Bridged2Bar12_Rounde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, Jumper:SolderJumper-3_P1.3mm_Bridged2Bar12_RoundedPad1.0x1.5mm, symbol lakemountain:SolderJumper_3_Bridged12
- added LOGO1: QMK Logo, lakemountain:QMK_PoweredBy, symbol lakemountain:Fiducial
- added LOGO2: OH Logo, lakemountain:OSHW-Logo2_9.8x8mm_SilkScreen, symbol lakemountain:Fiducial
- added R15: 10k, lakemountain:R_0603_1608Metric, symbol lakemountain:R-Device-keyboard-right-rescue
- added U10, U11, U9: SRV05-4, lakemountain:SOT-23-6, symbol lakemountain:SRV05-4
- C1, C11, C2, C3, C5, C6, C9: symbol Bonsai_C4:cap_100nF_16v_0402 -> lakemountain:cap_100nF_16v_0402
- C10: symbol Bonsai_C4:cap_10uF_10v_0402 -> lakemountain:cap_10uF_10v_0402
- C12, C7: symbol Bonsai_C4:cap_4.7uF_10v_0402 -> lakemountain:cap_4.7uF_10v_0402
- C13, C14, C15, C16, C17, C18, C19, C20, C21, C24, C25, C26, C27, C28, C29, C30, C31: symbol Device:C -> lakemountain:C
- C22, C23: symbol Bonsai_C4:cap_20pF_50v_0402 -> lakemountain:cap_20pF_50v_0402
- C4, C8: symbol Bonsai_C4:cap_1uF_10v_0402 -> lakemountain:cap_1uF_10v_0402
- D1: symbol YAEMK:LED -> lakemountain:LED
- D2: symbol Bonsai_C4:PMEG2010AEB -> lakemountain:PMEG2010AEB
- D3: symbol Bonsai_C4:SMD-LED-WHITE_0402_ -> lakemountain:SMD-LED-WHITE_0402_
- Da1, Da2, Da3, Da4, Da5, Da6, Da7, Da8, Db1, Db10, Db11, Db2, Db3, Db4, Db5, Db6, Db7, Db8, Db9, Dc1, Dc2, Dc3, Dc4, Dc5, Dc6, Dc7, Dd1, Dd2, Dd3, Dd4, Dd5, Dd6, Dd7, Dd8, De1, De2, De3, De4, De5, De6, De7: symbol Device:D -> lakemountain:D
- ENC1: symbol Djinn-rescue:Rotary_Encoder_Switch-Device -> lakemountain:Rotary_Encoder_Switch-Device; JLCPCB BOM (none) -> 0; now not fitted
- F1, F2: symbol Bonsai_C4:SMD-PPTC-500MA_0805_ -> lakemountain:SMD-PPTC-500MA_0805_
- FB1, FB2, FB3, FB4: symbol Bonsai_C4:fb_0402_26ohm -> lakemountain:fb_0402_26ohm
- H1, H2, H3: symbol Mechanical:MountingHole_Pad -> lakemountain:MountingHole_Pad
- J1, J3, J5, J6: symbol keyboard-left-rescue:USB_C_Receptacle_USB2.0-Connector-keyboard-right-rescue -> lakemountain:USB_C_Receptacle_USB2.0-Connector-keyboard-right-rescue
- J2: symbol Connector_Generic:Conn_01x06 -> lakemountain:Conn_01x06
- J4: symbol marbastlib-various:JTAG_TC2030 -> lakemountain:JTAG_TC2030
- JP3, JP4: symbol Jumper:SolderJumper_3_Open -> lakemountain:SolderJumper_3_Open
- LEDa1, LEDa2, LEDa3, LEDa4, LEDa5, LEDa6, LEDa7, LEDa8, LEDc1, LEDc2, LEDc3, LEDc4, LEDc5, LEDc6, LEDc8, LEDe1, LEDe2, LEDe3, LEDe4, LEDe5, LEDe6, LEDe7: footprint lakemountain:LED_MX_6028R -> marbastlib-mx:LED_MX_6028R; symbol keyboard-mx:MX_SK6812MINI-E -> lakemountain:MX_SK6812MINI-E
- LEDb1, LEDb2, LEDb3, LEDb4, LEDb5, LEDb6, LEDb7, LEDb8, LEDb9, LEDd1, LEDd2, LEDd3, LEDd4, LEDd5, LEDd8: footprint lakemountain:LED_MX_6028R_Flipped -> marbastlib-mx:LED_MX_6028R; symbol keyboard-mx:MX_SK6812MINI-E -> lakemountain:MX_SK6812MINI-E
- LEDc7: footprint lakemountain:LED_MX_6028R_SOLO -> marbastlib-mx:LED_MX_6028R; symbol keyboard-mx:MX_SK6812MINI-E -> lakemountain:MX_SK6812MINI-E
- LEDd6: symbol keyboard-mx:MX_SK6812MINI-E -> lakemountain:MX_SK6812MINI-E
- LEDd7: footprint lakemountain:LED_MX_6028R_Flipped -> lakemountain:LED_MX_6028R_SOLO; symbol keyboard-mx:MX_SK6812MINI-E -> lakemountain:MX_SK6812MINI-E
- LEDs1, LEDs10, LEDs11, LEDs12, LEDs13, LEDs14, LEDs15, LEDs16, LEDs17, LEDs18, LEDs19, LEDs2, LEDs3, LEDs4, LEDs5, LEDs6, LEDs7, LEDs8, LEDs9: footprint lakemountain:sk6812side -> marbastlib-mx:LED_MX_6028R; symbol keyboard-mx:MX_SK6812MINI-E -> lakemountain:MX_SK6812MINI-E
- LS1: symbol keyboard-left-rescue:Speaker-Device-keyboard-right-rescue -> lakemountain:Speaker-Device-keyboard-right-rescue
- Q1, Q2: symbol Bonsai_C4:MUN5311DW1T1G -> lakemountain:MUN5311DW1T1G
- Q3: symbol Transistor_FET:AO3401A -> lakemountain:AO3401A
- R1, R2, R3, R4, R6, R8: symbol keyboard-left-rescue:R-Device-keyboard-right-rescue -> lakemountain:R-Device-keyboard-right-rescue
- R10: symbol Bonsai_C4:r_4.7k_0402_1p -> lakemountain:r_4.7k_0402_1p
- R11: symbol Bonsai_C4:r_10k_0402_1p -> lakemountain:r_10k_0402_1p
- R12, R5: symbol Bonsai_C4:r_75_0402_1p -> lakemountain:r_75_0402_1p
- R13: symbol keyboard-left-rescue:R-Device-keyboard-right-rescue -> lakemountain:R-Device-keyboard-right-rescue; JLCPCB BOM 1 -> 0; now not fitted
- R14: symbol keyboard-left-rescue:R-Device-keyboard-right-rescue -> lakemountain:R-Device-keyboard-right-rescue; JLCPCB BOM 0 -> 1
- R7: symbol Bonsai_C4:r_100k_0402_1p -> lakemountain:r_100k_0402_1p
- R9: symbol Bonsai_C4:r_470_0402_1p -> lakemountain:r_470_0402_1p
- S1, S2: symbol marbastlib-mx:MX_stab -> lakemountain:MX_stab
- S3: footprint lakemountain:STAB_MX_P_ISO_FLIPPED -> lakemountain:STAB_MX_P_ISO; symbol marbastlib-mx:MX_stab -> lakemountain:MX_stab
- S4, S5: symbol marbastlib-mx:MX_stab -> lakemountain:MX_stab; JLCPCB BOM (none) -> 0; now not fitted
- SW1: symbol keyboard_parts:SW_PUSH -> lakemountain:SW_PUSH
- SWa1, SWa2, SWa3, SWa4, SWa5, SWa6, SWa7, SWa8, SWb1, SWb2, SWb3, SWb4, SWb5, SWb6, SWb7, SWb8, SWb9, SWc1, SWc2, SWc3, SWc4, SWc5, SWc6, SWc7, SWc8, SWd1, SWd2, SWd3, SWd4, SWd5, SWd6, SWd7, SWd8, SWe1, SWe2, SWe3, SWe4, SWe5, SWe6, SWe7: symbol keyboard-mx:MX_SW_HS -> lakemountain:MX_SW_HS
- SWbx8, SWcx7, SWd9, SWe10, SWe11, SWe8, SWe9: symbol keyboard-mx:MX_SW_HS -> lakemountain:MX_SW_HS; JLCPCB BOM (none) -> 0; now not fitted
- U1: symbol MCU_ST_STM32F4:STM32F411RETx -> lakemountain:STM32F411RETx
- U2: symbol Bonsai_C4:AAP2967-33VIR1 -> lakemountain:AAP2967-33VIR1
- U4: symbol Bonsai_C4:SRV05-4 -> lakemountain:SRV05-4
- U5: symbol Bonsai_C4:SN74LV1T34DCKR -> lakemountain:SN74LV1T34DCKR
- U6: symbol Amplifier_Operational:LMV321 -> lakemountain:LMV321
- U7: symbol Bonsai_C4:MB85RS64PNF-G-JNERE1 -> lakemountain:MB85RS64PNF-G-JNERE1
- U8: symbol Bonsai_C4:W25Q128JVSIQ -> lakemountain:W25Q128JVSIQ
- U9: symbol Analog_Switch:TS3A27518ERTW -> lakemountain:TS3A27518ERTW
- Y1: symbol Bonsai_C4:SMD-CRYSTAL-8MHZ-20PF-10PPM_2P-5.0X3.2MM_ -> lakemountain:SMD-CRYSTAL-8MHZ-20PF-10PPM_2P-5.0X3.2MM_
Connections:
- net x1 is gone; now on net SPI_MISO: U9.23 (NC1)
- net x2 is gone; now on net SPI_MOSI: U9.22 (NC2)
- net x3 is gone; now on net JTDO: U9.20 (NC3)
- net +3.3V: now also JP2.3 (B), JP6.3 (B), JP8.3 (B)
- net +5V: now also JP2.1 (A), JP8.1 (A)
- net CONN_CS: no longer J6.A8 (SBU1), J6.B8 (SBU2)
- net CONN_SEL: now also U1.39 (PC8), JP1.1 (A), R15.1
- net GND: now also JP6.1 (A), R15.2, U10.2 (VN), U11.2 (VN), U9.2 (VN)
- net SPI_MISO: now also U11.6 (IO4)
- net USART2_RX: now also U9.1 (IO1)
- net USART2_TX: now also U9.3 (IO2)
- net USB_VBUS_IN_LINK: now also U9.5 (VP)
- net col7: now also U1.37 (PC6)
- net col8: now also U1.38 (PC7)
- net z1: now also U10.4 (IO3)
- net z2: now also U10.1 (IO1)
- net z3: now also U10.3 (IO2)
- net z4: now also U10.6 (IO4)
- net at LEDs18.2 (DOUT): now also LEDs19.3 (DIN); no longer LEDs17.3 (DIN)
- net at LEDs18.3 (DIN): now also LEDs17.2 (DOUT); no longer LEDs19.2 (DOUT)
- net at LEDs14.2 (DOUT): now also LEDs12.3 (DIN)
- net at LEDs14.3 (DIN): now also LEDs19.2 (DOUT); no longer LEDs12.2 (DOUT)
- net at LEDd8.2 (DOUT): now also LEDc8.3 (DIN); no longer LEDd7.3 (DIN)
- net at LEDd8.3 (DIN): now also LEDe6.2 (DOUT); no longer LEDc8.2 (DOUT)
- net at LEDs10.2 (DOUT): now also LEDs8.3 (DIN); no longer LEDs12.3 (DIN)
- net at LEDs7.2 (DOUT): now also LEDs9.3 (DIN); no longer LEDs5.3 (DIN)
- net at LEDs7.3 (DIN): now also LEDs5.2 (DOUT); no longer LEDs9.2 (DOUT)
- net at LEDs10.3 (DIN): now also LEDs12.2 (DOUT); no longer LEDs8.2 (DOUT)
- net at LEDs6.2 (DOUT): no longer LEDs8.3 (DIN)
- net at LEDs16.2 (DOUT): now also LEDs17.3 (DIN); no longer LEDs15.3 (DIN)
- net at LEDs16.3 (DIN): now also LEDs15.2 (DOUT); no longer LEDs17.2 (DOUT)
- net at LEDs11.2 (DOUT): now also LEDs13.3 (DIN); no longer LEDs9.3 (DIN)
- net at J5.A4 (VBUS), J5.A9 (VBUS), J5.B4 (VBUS)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: now also JP8.2 (C), U10.5 (VP)
- net DO60: now reaches LEDe5.2 (DOUT), LEDe6.3 (DIN)
- net DO60: now also JP1.1 (A)
- net at LEDs3.2 (DOUT): now also LEDs2.3 (DIN); no longer LEDs4.3 (DIN)
- net at LEDs3.3 (DIN): now also LEDs4.2 (DOUT); no longer LEDs2.2 (DOUT)
- net at U9.11 (IN2), U9.21 (IN1): now also JP1.2 (C)
- net at LEDb9.2 (DOUT): now also LEDa8.3 (DIN); no longer LEDb8.3 (DIN)
- net at LEDb9.3 (DIN): now also LEDc8.2 (DOUT); no longer LEDa8.2 (DOUT)
- net at LEDs11.3 (DIN): now also LEDs9.2 (DOUT); no longer LEDs13.2 (DOUT)
- net at J6.A4 (VBUS), J6.A9 (VBUS), J6.B4 (VBUS)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: now also JP2.2 (C), U11.5 (VP)
- net at LEDa7.2 (DOUT): now also LEDb8.3 (DIN); no longer LEDa8.3 (DIN)
- net at LEDc7.2 (DOUT): now also LEDd7.3 (DIN); no longer LEDc8.3 (DIN)
- net at LEDs6.3 (DIN): now also LEDs8.2 (DOUT); no longer LEDs4.2 (DOUT)
- net at J6.A7 (D-), J6.B7 (D-), JP3.2 (C): now also U11.3 (IO2)
- net at LEDs1.2 (DOUT): now also LEDs5.3 (DIN); no longer LEDs2.3 (DIN)
- net at LEDs1.3 (DIN): now also LEDs2.2 (DOUT); no longer LEDs5.2 (DOUT)
- net at J6.A6 (D+), J6.B6 (D+), JP4.2 (C): now also U11.1 (IO1)
- new net: JP1.3 (B), JP6.2 (C)
- new net: LEDs13.2 (DOUT), LEDs15.3 (DIN)
- new net CONN2_CS: J6.A8 (SBU1), J6.B8 (SBU2), U11.4 (IO3)
- new net DO65: JP1.2 (B), LEDa8.2 (DOUT), LEDs4.3 (DIN)
- no-connect marks 28 -> 27
Other:
- note added: "Bridge if 60% layout"
- note added: "Pull down CONN_SEL for default 0"
- note removed: "Bridge JP8/JP9/JP10 if 60% layout"
- note removed: "Testpoints"
- moved on the sheet: C1, C10, C11, C13, C14, C15, C16, C17, C18, C19, C20, C21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

Commit message: Update right schematic symbols
Parts:
- C1, C10, C11, C12, C2, C22, C23, C3, C4, C5, C6, C7, C8, C9: footprint Bonsai_C4:C_0402_1005Metric -> lakemountain:C_0402_1005Metric
- C13, C14, C15, C16, C17, C18, C19, C20, C21, C24, C25, C26, C27, C28, C29, C30, C31: footprint Bonsai_C4:C_0805 -> lakemountain:C_0805
- D1: footprint LED_SMD:LED_0603_1608Metric -> lakemountain:LED_0603_1608Metric
- D2, De1: footprint Bonsai_C4:D_SOD-523 -> lakemountain:D_SOD-523
- D3: footprint Bonsai_C4:LED_0402 -> lakemountain:LED_0402
- Da1, Da2, Da3, Da4, Da5, Da6, Da7, Da8, Db1, Db10, Db11, Db2, Db3, Db4, Db5, Db6, Db7, Db8, Db9, Dc1, Dc2, Dc3, Dc4, Dc5, Dc6, Dc7, Dd1, Dd2, Dd3, Dd4, Dd5, Dd6, Dd7, Dd8, De2, De3, De4, De5, De6, De7: footprint Diode_SMD:D_SOD-123 -> lakemountain:D_SOD-123
- F1, F2: footprint Bonsai_C4:F1206 -> lakemountain:F1206
- FB1, FB2, FB3, FB4, R10, R11, R12, R5, R7, R9: footprint Bonsai_C4:R_0402_1005Metric -> lakemountain:R_0402_1005Metric
- H1, H2, H3: footprint MountingHole:MountingHole_2.2mm_M2_Pad_Via -> lakemountain:MountingHole_2.2mm_M2_Pad_Via
- J2: footprint Connector_PinHeader_2.54mm:PinHeader_1x06_P2.54mm_Vertical -> lakemountain:PinHeader_1x06_P2.54mm_Vertical
- J4: footprint marbastlib-various:CON_TC2030_outlined -> lakemountain:CON_TC2030_outlined
- JP1: footprint Jumper:SolderJumper-2_P1.3mm_Open_RoundedPad1.0x1.5mm -> lakemountain:SolderJumper-2_P1.3mm_Open_RoundedPad1.0x1.5mm
- JP2, JP8: footprint Jumper:SolderJumper-3_P1.3mm_Bridged2Bar12_RoundedPad1.0x1.5mm -> lakemountain:SolderJumper-3_P1.3mm_Bridged2Bar12_RoundedPad1.0x1.5mm
- JP3, JP4: footprint Jumper:SolderJumper-3_P1.3mm_Open_RoundedPad1.0x1.5mm_NumberLabels -> lakemountain:SolderJumper-3_P1.3mm_Open_RoundedPad1.0x1.5mm_NumberLabels
- LEDa1, LEDa2, LEDa3, LEDa4, LEDa5, LEDa6, LEDa7, LEDa8, LEDc1, LEDc2, LEDc3, LEDc4, LEDc5, LEDc6, LEDc7, LEDc8, LEDe1, LEDe2, LEDe3, LEDe4, LEDe5, LEDe6, LEDe7: footprint marbastlib-mx:LED_MX_6028R -> lakemountain:LED_MX_6028R
- LEDb1, LEDb2, LEDb3, LEDb4, LEDb5, LEDb6, LEDb7, LEDb8, LEDb9, LEDd1, LEDd2, LEDd3, LEDd4, LEDd5, LEDd8: footprint marbastlib-mx:LED_MX_6028R -> lakemountain:LED_MX_6028R_Flipped
- LEDs1, LEDs10, LEDs11, LEDs12, LEDs13, LEDs14, LEDs15, LEDs16, LEDs17, LEDs18, LEDs19, LEDs2, LEDs3, LEDs4, LEDs5, LEDs6, LEDs7, LEDs8, LEDs9: footprint marbastlib-mx:LED_MX_6028R -> lakemountain:sk6812side
- Q1, Q2: footprint Bonsai_C4:SOT-363_SC-70-6_SC-88 -> lakemountain:SOT-363_SC-70-6_SC-88
- Q3: footprint Package_TO_SOT_SMD:SOT-23 -> lakemountain:SOT-23
- R1: footprint Resistor_SMD:R_0805_2012Metric_Pad1.20x1.40mm_HandSolder -> lakemountain:R_0805_2012Metric_Pad1.20x1.40mm_HandSolder
- R13, R14, R2, R3, R4, R6, R8: footprint Resistor_SMD:R_0603_1608Metric -> lakemountain:R_0603_1608Metric
- SW1: footprint Button_Switch_SMD:SW_SPST_TL3342 -> lakemountain:SW_SPST_TL3342
- U1: footprint Package_QFP:LQFP-64_10x10mm_P0.5mm -> lakemountain:LQFP-64_10x10mm_P0.5mm
- U2: footprint Bonsai_C4:SOT-23-5 -> lakemountain:SOT-23-5
- U4: footprint Bonsai_C4:SOT-23-6 -> lakemountain:SOT-23-6
- U5: footprint Bonsai_C4:SOT-353_SC-70-5 -> lakemountain:SOT-353_SC-70-5
- U6: footprint Package_TO_SOT_SMD:SOT-23-5 -> lakemountain:SOT-23-5
- U7: footprint Bonsai_C4:SOP-8_3.9x4.9mm_P1.27mm -> lakemountain:SOP-8_3.9x4.9mm_P1.27mm
- U8: footprint Bonsai_C4:SOIC-8_5.23x5.23mm_P1.27mm -> lakemountain:SOIC-8_5.23x5.23mm_P1.27mm
- Y1: footprint Bonsai_C4:X2-SMD-5.0X3.2X1.3MM -> lakemountain:X2-SMD-5.0X3.2X1.3MM

Commit message: Push latest, don't remember changes...
Parts:
- added LOGO1: Lakemountain Logo, lakemountain:LOGO, symbol lakemountain:Fiducial
- added LOGO1: QR, lakemountain:QR_Code, symbol lakemountain:Fiducial
- J2: now not fitted
Connections:
- net JOY_X is gone; now on net CONN2_CS: U1.2 (PC13)
- net ENC_2_A: no longer names the net of U1.40 (PC9)
- net ENC_2_B: no longer names the net of U1.51 (PC10)
- no-connect marks 27 -> 29
Other:
- moved on the sheet: C22, C23, LOGO1, LOGO2, R13, R14, Y1
